Commit message: add RC26_zhangai.world

File: livox_laser_simulation_RO2/urdf/my_robot/plugins/gazebo_sensor_plugin.xacro (robot description, xacro)
@@ -46,6 +46,6 @@
                         <mean>0.0</mean>
                         <stddev>1.7e-2</stddev>
-                        <bias_mean>0.1</bias_mean>
-                        <bias_stddev>0.001</bias_stddev>
+                        <bias_mean>0.0</bias_mean>
+                        <bias_stddev>0.0001</bias_stddev>
                     </noise>
                 </x>
@@ -54,6 +54,6 @@
                         <mean>0.0</mean>
                         <stddev>1.7e-2</stddev>
-                        <bias_mean>0.1</bias_mean>
-                        <bias_stddev>0.001</bias_stddev>
+                        <bias_mean>0.0</bias_mean>
+                        <bias_stddev>0.0001</bias_stddev>
                     </noise>
                 </y>
@@ -62,6 +62,6 @@
                         <mean>0.0</mean>
                         <stddev>1.7e-2</stddev>
-                        <bias_mean>0.1</bias_mean>
-                        <bias_stddev>0.001</bias_stddev>
+                        <bias_mean>0.0</bias_mean>
+                        <bias_stddev>0.0001</bias_stddev>
                     </noise>
                 </z>

File: livox_laser_simulation_RO2/urdf/my_robot/sensor/mid360.xacro (robot description, xacro)
@@ -4,8 +4,8 @@
   <xacro:property name="laser_min_range" value="0.1"/>
   <xacro:property name="laser_max_range" value="200.0"/>
-  <xacro:property name="samples" value="30000"/>
-  <xacro:property name="resolution" value="0.002"/>
+  <xacro:property name="samples" value="40000"/>
+  <xacro:property name="resolution" value="0.0015"/>
   <xacro:property name="noise_mean" value="0.0"/>
-  <xacro:property name="noise_stddev" value="0.002"/>
+  <xacro:property name="noise_stddev" value="0.0015"/>
   <xacro:property name="mass" value="0.4" />
   <xacro:property name="length" value="0.1" />
