Commit message: add RC26_zhangai.world && RC26_renwu.world

File: livox_laser_simulation_RO2/urdf/my_robot/plugins/gazebo_control_plugin.xacro (robot description, xacro)
@@ -3,57 +3,50 @@
    <!-- 按需更改 名字 -->
     <xacro:macro name="my_robot_ros2_control_planar">
-        <ros2_control name="MyRobotPlanarSystem" type="system">
+        <ros2_control name="MyRobotSystem" type="system">
             <hardware>
                 <plugin>gazebo_ros2_control/GazeboSystem</plugin>
             </hardware>
+            <joint name="ahead_left_wheel_joint">
+                <command_interface name="velocity">
+                    <param name="min">-30.0</param>
+                    <param name="max">30.0</param>
+                </command_interface>
+                <state_interface name="position"/>
+                <state_interface name="velocity"/>
+            </joint>
+            <joint name="ahead_right_wheel_joint">
+                <command_interface name="velocity">
+                    <param name="min">-30.0</param>
+                    <param name="max">30.0</param>
+                </command_interface>
+                <state_interface name="position"/>
+                <state_interface name="velocity"/>
+            </joint>
+            <joint name="bhind_left_wheel_joint">
+                <command_interface name="velocity">
+                    <param name="min">-30.0</param>
+                    <param name="max">30.0</param>
+                </command_interface>
+                <state_interface name="position"/>
+                <state_interface name="velocity"/>
+            </joint>
+            <joint name="bhind_right_wheel_joint">
+                <command_interface name="velocity">
+                    <param name="min">-30.0</param>
+                    <param name="max">30.0</param>
+                </command_interface>
+                <state_interface name="position"/>
+                <state_interface name="velocity"/>
+            </joint>
         </ros2_control>
         <gazebo>
-        <!-- libgazebo_ros_planar_move.so 是 平面移动插件 -->
-            <plugin name="planar_move" filename="libgazebo_ros_planar_move.so">
+            <plugin name="gazebo_ros2_control" filename="libgazebo_ros2_control.so">
                 <ros>
-                    <namespace>/</namespace>
-                    <remapping>cmd_vel:=cmd_vel</remapping>
-                    <remapping>odom:=odom</remapping>
+                    <remapping>diff_drive_controller/cmd_vel_unstamped:=cmd_vel</remapping>
+                    <remapping>diff_drive_controller/odom:=odom</remapping>
                 </ros>
-                <!-- 频率 -->
-                <update_rate>30</update_rate>
-                <!-- 里程计frame id -->
-                <odometry_frame>odom</odometry_frame>
-                  <!-- 是否发布里程计 -  -->
-                <publish_odom>true</publish_odom>
-                <!-- 是否发布里程计tf -->
-                <publish_odom_tf>true</publish_odom_tf>
-                <robot_base_frame>base_footprint</robot_base_frame>
-                <!-- 最大速度 -->
-                <max_vel_x>5.0</max_vel_x>
-                <max_vel_y>5.0</max_vel_y>
-                <max_vel_theta>3.14</max_vel_theta>
-                <!-- 最大加速度 -->
-                <max_accel_x>3.0</max_accel_x>
-                <max_accel_y>3.0</max_accel_y>
-                <max_accel_theta>3.14</max_accel_theta>
+                <parameters>$(find ros2_livox_simulation)/config/myrobot_ros2_controller.yaml</parameters>
             </plugin>
         </gazebo>
     </xacro:macro>
 </robot>
-<!-- <?xml version="1.0"?>
-<robot xmlns:xacro="http://www.ros.org/wiki/xacro">
-    <xacro:macro name="gazebo_planar_control_plugin">
-        <gazebo>
-            <plugin name="planar_move" filename="libgazebo_ros_planar_move.so">
-                <ros>
-                    <namespace>/</namespace>
-                    <remapping>cmd_vel:=cmd_vel</remapping>
-                </ros>
-                <update_rate>30</update_rate>
-                <publish_odom>false</publish_odom>
-                <publish_odom_tf>false</publish_odom_tf>
-                <robot_base_frame>base_footprint</robot_base_frame>
-                <max_vel_x>1.0</max_vel_x>
-                <max_vel_y>1.0</max_vel_y>
-                <max_vel_theta>1.57</max_vel_theta>
-            </plugin>
-        </gazebo>
-    </xacro:macro>
-</robot>
- -->

File: livox_laser_simulation_RO2/urdf/my_robot/sensor/mid360.xacro (robot description, xacro)
@@ -24,5 +24,5 @@
         <origin xyz="0.025 -0.0265 -0.025" rpy="${pi/2} 0 ${pi}"/>
         <geometry>
-          <mesh filename="package://ros2_livox_simulation/meshes/mid360.stl" scale="0.0008 0.0008 0.0008"/>
+          <mesh filename="file://$(find ros2_livox_simulation)/meshes/mid360.stl" scale="0.0008 0.0008 0.0008"/>
         </geometry>
       </visual>
@@ -30,5 +30,5 @@
     <origin xyz="0.025 -0.0265 -0.025" rpy="${pi/2} 0 ${pi}"/>
     <geometry>
-      <mesh filename="package://ros2_livox_simulation/meshes/mid360.stl" scale="0.0008 0.0008 0.0008"/>
+      <mesh filename="file://$(find ros2_livox_simulation)/meshes/mid360.stl" scale="0.0008 0.0008 0.0008"/>
     </geometry>
   </collision>
